File: hardware/hardware.kicad_sch (KiCad schematic)
At the start: 0 parts

Commit message: Completed Schematic
Parts:
- added C1: 0.47 uF, symbol Device:C_Polarized
- added C2: 33 uF, symbol Device:C_Polarized
- added C3: .1 uF, symbol Device:C
- added C4, C7: 1 uF, symbol Device:C
- added C5, C6, C8: 10 uF, symbol Device:C
- added D1: LED_RED, symbol Device:LED
- added D2: LED_GREEN, symbol Device:LED
- added R1, R2: 220 R, symbol Device:R
- added SW1: SW_SPST, symbol Switch:SW_SPST
- added U1: DHT11, Sensor:Aosong_DHT11_5.5x12.0_P2.54mm, symbol Sensor:DHT11
- added U2: SCD41, symbol ATDLib:SCD41
- added U3: ESP32 S3 WROOM1, symbol ATDLib:ESP32_S3_WROOM1
- added U4: PMS7003, symbol ATDLib:PMS7003
- added U5: LM3940, symbol ATDLib:LM3940
- added U6: MQ-135, symbol ATDLib:MQ-135
Connections:
- new net: SW1.1 (A), U3.1 (GND)
- new net: SW1.2 (B), U3.10 (5)
- new net: D2.1 (K), R2.1
- new net: D1.1 (K), R1.1
- new net +3.3V: C2.1, U3.6 (3v3), U5.3 (VCC_OUT)
- new net +5V: C1.1, C3.1, C4.1, C5.1, C6.1, C7.1, C8.1, U1.1 (VDD), U2.2 (VCC), U4.2 (VCC), U5.2 (VCC_IN), U6.2 (VCC)
- new net GND: C1.2, C2.2, C3.2, C4.2, C5.2, C6.2, C7.2, C8.2, R1.2, R2.2, U1.4 (GND), U2.1 (GND), U3.2 (GND), U4.1 (GND), U5.1 (GND), U6.1 (GND)
- new net GPIO 17: U3.15 (17), U4.4 (RX)
- new net GPIO 18: U3.16 (18), U4.5 (TX)
- new net GPIO 4: U1.2 (DATA), U3.9 (4)
- new net GPIO 6: D1.2 (A), U3.11 (6)
- new net GPIO 7: D2.2 (A), U3.12 (7)
- new net GPIO 8: U2.4 (SDA), U3.17 (8)
- new net GPIO 9: U2.3 (SCL), U3.20 (9)
- new net GPIO10: U3.21 (10), U6.3 (AO)
- new net GPIO11: U3.22 (11), U6.4 (DO)
- no-connect marks 0 -> 33
Other:
- company: (none) -> Serive
- title: (none) -> Air Tracking Device
